File: Esquematico_Luva.kicad_sch (KiCad schematic)
At the start: 12 parts, among them J1 9V Input, J2 Push Button, J3 Goniometer, J4 MPU6050, J5 Flex Sensor, U1 L7805, U2 ESP32-DEVKIT-V1

Commit message: feat(.kicad_sch): att project
Parts:
- gave numbers to parts that had none: 1
- renumbered J3 to J2, J2 to J3, J5 to J4, J4 to J6
Connections:
- no-connect marks 17 -> 21

Commit message: feat(sch): att libraries
Parts:
- C1, C2: footprint (none) -> Capacitor_THT:C_Disc_D5.1mm_W3.2mm_P5.00mm
- J1, J3, J4, J5: footprint (none) -> TerminalBlock:TerminalBlock_bornier-2_P5.08mm
- J2: footprint (none) -> TerminalBlock:TerminalBlock_bornier-3_P5.08mm
- J6: footprint (none) -> TerminalBlock:TerminalBlock_bornier-4_P5.08mm
- R1, R2: footprint (none) -> Resistor_THT:R_Axial_DIN0207_L6.3mm_D2.5mm_P10.16mm_Horizontal
- U1: footprint (none) -> footprints:TO255P1040X460X1968-3
- U2: footprint MODULE_ESP32_DEVKIT_V1 -> footprints:ESP32_DEV
Changed lines of the file:
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@@
     (property "Reference" "J2" (id 0) (at 35.56 77.47 0))
     (property "Value" "Goniometer" (id 1) (at 35.56 80.01 0))
-    (property "Footprint" "" (id 2) (at 39.37 74.93 0)
+    (property "Footprint" "TerminalBlock:TerminalBlock_bornier-3_P5.08mm" (id 2) (at 39.37 74.93 0)
       (effects (font (size 1.27 1.27)) hide)
     )
@@
     (property "Reference" "U1" (id 0) (at 48.26 27.94 0))
     (property "Value" "L7805" (id 1) (at 48.26 30.48 0))
-    (property "Footprint" "" (id 2) (at 48.895 39.37 0)
+    (property "Footprint" "footprints:TO255P1040X460X1968-3" (id 2) (at 48.895 39.37 0)
       (effects (font (size 1.27 1.27) italic) (justify left) hide)
     )
@@
       (effects (font (size 1.27 1.27)) (justify left))
     )
-    (property "Footprint" "" (id 2) (at 60.6552 43.18 0)
+    (property "Footprint" "Capacitor_THT:C_Disc_D5.1mm_W3.2mm_P5.00mm" (id 2) (at 60.6552 43.18 0)
       (effects (font (size 1.27 1.27)) hide)
     )
@@
     (property "Reference" "J4" (id 0) (at 35.56 119.38 0))
     (property "Value" "Flex Sensor" (id 1) (at 35.56 121.92 0))
-    (property "Footprint" "" (id 2) (at 39.37 116.84 0)
+    (property "Footprint" "TerminalBlock:TerminalBlock_bornier-2_P5.08mm" (id 2) (at 39.37 116.84 0)
       (effects (font (size 1.27 1.27)) hide)
     )
@@
     (property "Reference" "J1" (id 0) (at 17.78 38.1 0))
     (property "Value" "9V Input" (id 1) (at 17.78 40.64 0))
-    (property "Footprint" "" (id 2) (at 21.59 35.56 0)
+    (property "Footprint" "TerminalBlock:TerminalBlock_bornier-2_P5.08mm" (id 2) (at 21.59 35.56 0)
       (effects (font (size 1.27 1.27)) hide)
     )
@@
       (effects (font (size 1.27 1.27)) (justify left))
     )
-    (property "Footprint" "" (id 2) (at 37.7952 43.18 0)
+    (property "Footprint" "Capacitor_THT:C_Disc_D5.1mm_W3.2mm_P5.00mm" (id 2) (at 37.7952 43.18 0)
       (effects (font (size 1.27 1.27)) hide)
     )
@@
     (property "Reference" "R2" (id 0) (at 49.53 124.46 90))
     (property "Value" "10k" (id 1) (at 52.07 121.92 90))
-    (property "Footprint" "" (id 2) (at 50.8 121.158 90)
+    (property "Footprint" "Resistor_THT:R_Axial_DIN0207_L6.3mm_D2.5mm_P10.16mm_Horizontal" (id 2) (at 50.8 121.158 90)
       (effects (font (size 1.27 1.27)) hide)
     )
@@
     (property "Reference" "J3" (id 0) (at 35.56 93.98 0))
     (property "Value" "Push Button" (id 1) (at 35.56 96.52 0))
-    (property "Footprint" "" (id 2) (at 39.37 91.44 0)
+    (property "Footprint" "TerminalBlock:TerminalBlock_bornier-2_P5.08mm" (id 2) (at 39.37 91.44 0)
       (effects (font (size 1.27 1.27)) hide)
     )
@@
       (effects (font (size 1.27 1.27)) (justify left))
     )
-    (property "Footprint" "" (id 2) (at 177.8 58.42 0)
+    (property "Footprint" "TerminalBlock:TerminalBlock_bornier-4_P5.08mm" (id 2) (at 177.8 58.42 0)
       (effects (font (size 1.27 1.27)) hide)
     )
@@
     (property "Reference" "J5" (id 0) (at 81.28 38.1 0))
     (property "Value" "5V Input" (id 1) (at 81.28 40.64 0))
-    (property "Footprint" "" (id 2) (at 77.47 35.56 0)
+    (property "Footprint" "TerminalBlock:TerminalBlock_bornier-2_P5.08mm" (id 2) (at 77.47 35.56 0)
       (effects (font (size 1.27 1.27)) hide)
     )
@@
     (property "Reference" "U2" (id 0) (at 146.05 38.1 0))
     (property "Value" "ESP32-DEVKIT-V1" (id 1) (at 146.05 40.64 0))
-    (property "Footprint" "MODULE_ESP32_DEVKIT_V1" (id 2) (at 147.32 96.52 0)
+    (property "Footprint" "footprints:ESP32_DEV" (id 2) (at 147.32 96.52 0)
       (effects (font (size 1.27 1.27)) (justify bottom) hide)
     )
@@
     (property "Reference" "R1" (id 0) (at 49.53 99.06 90))
     (property "Value" "5,6k" (id 1) (at 52.07 96.52 90))
-    (property "Footprint" "" (id 2) (at 50.8 95.758 90)
+    (property "Footprint" "Resistor_THT:R_Axial_DIN0207_L6.3mm_D2.5mm_P10.16mm_Horizontal" (id 2) (at 50.8 95.758 90)
       (effects (font (size 1.27 1.27)) hide)
     )
@@
     )
     (path "/7151ec7f-2485-4daa-b28b-8fa43343322a"
-      (reference "C1") (unit 1) (value "0.33uF") (footprint "")
+      (reference "C1") (unit 1) (value "0.33uF") (footprint "Capacitor_THT:C_Disc_D5.1mm_W3.2mm_P5.00mm")
     )
     (path "/242b0568-cc03-4c80-917c-105c7503fc0a"
-      (reference "C2") (unit 1) (value "0.1uF") (footprint "")
+      (reference "C2") (unit 1) (value "0.1uF") (footprint "Capacitor_THT:C_Disc_D5.1mm_W3.2mm_P5.00mm")
     )
     (path "/293ea053-039f-44e6-8ab1-d5862424cdc8"
-      (reference "J1") (unit 1) (value "9V Input") (footprint "")
+      (reference "J1") (unit 1) (value "9V Input") (footprint "TerminalBlock:TerminalBlock_bornier-2_P5.08mm")
     )
     (path "/04e1e20f-0a00-470a-a59b-6648fff613be"
-      (reference "J2") (unit 1) (value "Goniometer") (footprint "")
+      (reference "J2") (unit 1) (value "Goniometer") (footprint "TerminalBlock:TerminalBlock_bornier-3_P5.08mm")
     )
     (path "/9e512f8f-98a7-4d74-9808-b3c1df066b95"
-      (reference "J3") (unit 1) (value "Push Button") (footprint "")
+      (reference "J3") (unit 1) (value "Push Button") (footprint "TerminalBlock:TerminalBlock_bornier-2_P5.08mm")
     )
     (path "/28896f99-ffbb-45d6-83e3-37c69c277991"
-      (reference "J4") (unit 1) (value "Flex Sensor") (footprint "")
+      (reference "J4") (unit 1) (value "Flex Sensor") (footprint "TerminalBlock:TerminalBlock_bornier-2_P5.08mm")
     )
     (path "/bc30b629-9b03-4aed-9604-6bf61d9ff845"
-      (reference "J5") (unit 1) (value "5V Input") (footprint "")
+      (reference "J5") (unit 1) (value "5V Input") (footprint "TerminalBlock:TerminalBlock_bornier-2_P5.08mm")
     )
     (path "/a65c1eac-92c8-459f-905f-a8c4d4622922"
-      (reference "J6") (unit 1) (value "MPU6050") (footprint "")
+      (reference "J6") (unit 1) (value "MPU6050") (footprint "TerminalBlock:TerminalBlock_bornier-4_P5.08mm")
     )
     (path "/d274f6d8-44bf-4136-8c5c-46253f9cd17a"
-      (reference "R1") (unit 1) (value "5,6k") (footprint "")
+      (reference "R1") (unit 1) (value "5,6k") (footprint "Resistor_THT:R_Axial_DIN0207_L6.3mm_D2.5mm_P10.16mm_Horizontal")
     )
     (path "/7cc8864f-d444-4027-8ec9-21c2d8f61d5e"
-      (reference "R2") (unit 1) (value "10k") (footprint "")
+      (reference "R2") (unit 1) (value "10k") (footprint "Resistor_THT:R_Axial_DIN0207_L6.3mm_D2.5mm_P10.16mm_Horizontal")
     )
     (path "/0ec8662e-b2a9-40a2-ad8c-60814485e09d"
-      (reference "U1") (unit 1) (value "L7805") (footprint "")
+      (reference "U1") (unit 1) (value "L7805") (footprint "footprints:TO255P1040X460X1968-3")
     )
     (path "/c1fd6def-684b-4811-add8-d9a8e29fdb6d"
-      (reference "U2") (unit 1) (value "ESP32-DEVKIT-V1") (footprint "MODULE_ESP32_DEVKIT_V1")
-    )
-  )
+      (reference "U2") (unit 1) (value "ESP32-DEVKIT-V1") (footprint "footprints:ESP32_DEV")
+    )
+  )
